Commit message: Cleaned up some of the mess

File: hrl_gazebo_autobed/urdf/autobed_v2.URDF (robot description, URDF)
Before this commit: robot autobed, 10 links, 9 joints
Links:
- removed link torso_lift_link
- removed link world
- added link bed_frame_link, mass 128.981; collision mesh filename=package://bed_and_body_v4/meshes/bed_frame_link.STL; visual mesh filename=package://bed_and_body_v4/meshes/bed_frame_link.STL
- link base_link: mass 582.60172808288 -> 5.8260172808288; geometry collision mesh filename=package://bed_and_body_v4/meshes/base_link.STL; visual mesh filename=package://bed_and_body_v4/meshes/base_link.STL
- link head_rest_link: mass 5.2153755040103 -> 46.745755040103; geometry collision mesh filename=package://bed_and_body_v4/meshes/head_rest_link.STL; visual mesh filename=package://bed_and_body_v4/meshes/head_rest_link.STL
- link head_rest_spring: mass 10.0 -> 105.408; geometry collision mesh filename=package://bed_and_body_v4/meshes/head_rest_spring.STL; visual mesh filename=package://bed_and_body_v4/meshes/head_rest_spring.STL
- link leg_rest_lower_link: mass 3.25835 -> 31.5675; geometry collision mesh filename=package://bed_and_body_v4/meshes/leg_rest_lower_link.STL; visual mesh filename=package://bed_and_body_v4/meshes/leg_rest_lower_link.STL
- link leg_rest_lower_spring: mass 10.016 -> 101.016; geometry collision mesh filename=package://bed_and_body_v4/meshes/leg_rest_lower_spring.STL; visual mesh filename=package://bed_and_body_v4/meshes/leg_rest_lower_spring.STL
- link leg_rest_upper_link: mass 02.10955 -> 16.9275; geometry collision mesh filename=package://bed_and_body_v4/meshes/leg_rest_upper_link.STL; visual mesh filename=package://bed_and_body_v4/meshes/leg_rest_upper_link.STL
- link leg_rest_upper_spring: mass 5.0 -> 54.168; geometry collision mesh filename=package://bed_and_body_v4/meshes/leg_rest_upper_spring.STL; visual mesh filename=package://bed_and_body_v4/meshes/leg_rest_upper_spring.STL
- link mid_body_link: mass 4.0992 -> 40.992; geometry collision mesh filename=package://bed_and_body_v4/meshes/mid_body_link.STL; visual mesh filename=package://bed_and_body_v4/meshes/mid_body_link.STL
Joints:
- removed joint X
- removed joint autobed_height_joint
- removed joint mid_body_support
- added joint mid_body_link: type fixed, parent bed_frame_link, child mid_body_link, origin xyz=0.782663137625778 0 0.0499999999999999 rpy=1.5707963267949 -8.02446817831858E-32 -1.5707963267949, axis 0 0 0
- added joint tele_legs_joint: type prismatic, parent base_link, child bed_frame_link, origin xyz=-0.02 0 0.280500000000001 rpy=0 0 0, axis 0 0 -1
- joint head_rest_hinge: axis 0 0 1 -> 0 -1 0; limit lower=0 upper=1.57 effort=2000 velocity=0.2 -> lower=0 upper=1.57 effort=0 velocity=0; origin xyz=0.775 0 0.26 rpy=1.5708 1.0561E-10 3.1416 -> xyz=0 0.21 0 rpy=1.5708 1.5708 0
- joint leg_rest_upper_joint: limit lower=0 upper=1 effort=2000 velocity=0.2 -> lower=0 upper=1 effort=0 velocity=0
- joint leg_rest_upper_lower_joint: axis 0 0 1 -> 0 -1 0; limit lower=0 upper=0 effort=0 velocity=0 -> effort=0 velocity=0; origin xyz=0.37 0 0 rpy=-3.7123E-16 5.9121E-16 3.7854E-11 -> xyz=0.34869 0 0.12375 rpy=0 0 0
