Commit message: First working model of the two layered bed structure: The URDF to SDF conversion is not working. Will have to convert fixed joints to revolute with 0 limits

File: hrl_gazebo_autobed/urdf/autobed_template.URDF (robot description, URDF)
Before this commit: robot autobed, 10 links, 9 joints
Joints:
- joint head_rest_hinge: axis 0 1 0 -> 0 0 1; origin xyz=0 0.21 0 rpy=0 1.57 1.57 -> xyz=0.775 0 0.26 rpy=1.5708 1.0561E-10 3.1416
- joint leg_rest_upper_joint: origin xyz=0 0.21 -0.28 rpy=0 1.5708 1.5708 -> xyz=0 0.21 -0.28 rpy=1.5708 1.5708 0
- joint leg_rest_upper_lower_joint: axis 0 -1 0 -> 0 0 1; origin xyz=0.37 0 0 rpy=0 0 0 -> xyz=0.37 0 0 rpy=-3.7123E-16 5.9121E-16 3.7854E-11
- joint mid_body_support: origin xyz=0.78266 0 0.05 rpy=1.5708 -8.0245E-32 -1.5708 -> xyz=0.782663137625778 0 0.0499999999999999 rpy=1.5707963267949 -8.02446817831858E-32 -1.5707963267949
