Commit message: Gazebo model of Autobed tested and working v.1.1

File: hrl_gazebo_autobed/urdf/autobed.URDF (robot description, URDF)
Before this commit: robot autobed, 6 links, 5 joints
Joints:
- joint head_rest_hinge: limit lower=0 upper=1.057 effort=0 velocity=0 -> lower=0 upper=1.057 effort=2000 velocity=0.2
- joint leg_rest_upper_joint: limit lower=0 upper=1 effort=0 velocity=0 -> lower=0 upper=1 effort=2000 velocity=0.2

Commit message: Working tactile sensor for head rest

File: hrl_gazebo_autobed/urdf/autobed.URDF (robot description, URDF)
Before this commit: robot autobed, 6 links, 5 joints
Links:
- removed link bed_frame_link
- added link torso_lift_link, mass 18.2783; collision mesh filename=package://hrl_gazebo_autobed/urdf/meshes/torso_lift_link.STL; visual mesh filename=package://hrl_gazebo_autobed/urdf/meshes/torso_lift_link.STL
Joints:
- joint autobed_height_joint: child bed_frame_link -> torso_lift_link
- joint head_rest_hinge: parent bed_frame_link -> torso_lift_link
- joint leg_rest_upper_joint: parent bed_frame_link -> torso_lift_link

Commit message: Ironed out the errors from pose estimation pressure mapping engine

File: hrl_gazebo_autobed/urdf/autobed.URDF (robot description, URDF)
Before this commit: robot autobed, 6 links, 5 joints
Joints:
- joint leg_rest_upper_lower_joint: type fixed -> revolute

Commit message: Working multilayered autobed. Still takes time for the pressure map to be generated and updated.

File: hrl_gazebo_autobed/urdf/autobed.URDF (robot description, URDF)
Before this commit: robot autobed, 10 links, 9 joints
Joints:
- joint head_support: axis 0 0 0 -> 0 0 1; limit (none) -> lower=0 upper=0 effort=0 velocity=0; type fixed -> revolute
- joint leg_rest_lower_support: axis 0 0 0 -> 0 0 1; limit (none) -> lower=0 upper=0 effort=0 velocity=0; type fixed -> revolute
- joint leg_rest_upper_support: axis 0 0 0 -> 0 0 1; limit (none) -> lower=0 upper=0 effort=0 velocity=0; type fixed -> revolute
- joint mid_body_support: axis 0 0 0 -> 0 0 1; limit (none) -> lower=0 upper=0 effort=0 velocity=0; type fixed -> revolute

Commit message: Working autobed with gazebo version imitating physical. Lower leg link is like physical beds

File: hrl_gazebo_autobed/urdf/autobed.URDF (robot description, URDF)
Before this commit: robot autobed, 10 links, 9 joints
Joints:
- joint leg_rest_upper_lower_joint: limit lower=0 upper=0 effort=0 velocity=0 -> lower=-0.785 upper=0 effort=2000 velocity=0.2

Commit message: Added RVIZ stuff and tested with pose estimation. Basic results working

File: hrl_gazebo_autobed/urdf/autobed.URDF (robot description, URDF)
Before this commit: robot autobed, 10 links, 9 joints
Links:
- added link camera_link
Joints:
- added joint torso_camera_joint: type fixed, parent world, child camera_link, origin xyz=1.52 1.35 1.33 rpy=0.03 0.5 -3.0
- joint X: origin xyz=1.07 -1.1433776843867E-16 0.0 rpy=0 0 0 -> xyz=0.0 -1.1433776843867E-16 0.0 rpy=0 0 1.57079632679

Commit message: Fixed some bugs in the RViz so that bed height actuator resembles physical bed

File: hrl_gazebo_autobed/urdf/autobed.URDF (robot description, URDF)
Before this commit: robot autobed, 11 links, 10 joints
Joints:
- joint autobed_height_joint: limit lower=0.09 upper=0.2 effort=2000 velocity=0.2 -> lower=0.0 upper=0.2 effort=2000 velocity=0.2

Commit message: Added functionality for RVIZ to dynamically adjust for Kinect position: The Kinect is equipped with a marker cluster on its head, this is given the name camera_o. Our code subscribes to camera_o/pose and updates rviz viewpoint to match that of the correct position of the kinect.

File: hrl_gazebo_autobed/urdf/autobed.URDF (robot description, URDF)
Before this commit: robot autobed, 11 links, 10 joints
Links:
- removed link camera_link
Joints:
- removed joint torso_camera_joint
